File: hardware/rev0/luna_rev0.kicad_pcb (KiCad board)
At the start: 4 copper layers, 48 x 48 mm, 202 parts, among them IC1 ECP5-BGA256, J1 USB_C_Receptacle_USB2.0, J10 TC_SWD, J11 PMOD_B, J2 USB_C_Receptacle_USB2.0, J3 USB_A, J4 USB_C_Receptacle_USB2.0, J5 Conn_FPGA_JTAG_10, J6 Conn_ARM_JTAG_SWD_10, J7 PMOD_A, J8 Conn_Coaxial, J9 Conn_Coaxial, SW1 BTN_DFU, SW2 BTN_RESET, U1 AP22811A, U10 HyperRAM, U11 USB3343, U12 AP22811A, U13 AP22811A, U14 74AUP2G126, U2 74AUP2G126, U3 AP7366-33W5-7, U4 TCR2EF115, U5 MIC5504-2.5YM5, U6 ATSAMD11D14A-MUT, U7 W25Q32JVSS, U8 USB3343, U9 USB3343, Y1 Osc60MHz

Commit message: updated to kicad nightly
Connections:
- net /FPGA Configuration and Dev Features/~CS_DI renamed /FPGA Configuration and Dev Features/~{CS_DI}
- net /FPGA Configuration and Dev Features/~FORCE_DFU renamed /FPGA Configuration and Dev Features/~{FORCE_DFU}
- net /FPGA Configuration and Dev Features/~FPGA_INIT renamed /FPGA Configuration and Dev Features/~{FPGA_INIT}
- net /FPGA Configuration and Dev Features/~FPGA_PROGRAM renamed /FPGA Configuration and Dev Features/~{FPGA_PROGRAM}
- net /FPGA Configuration and Dev Features/~FPGA_SELF_PROGRAM renamed /FPGA Configuration and Dev Features/~{FPGA_SELF_PROGRAM}
- net /FPGA Configuration and Dev Features/~SIDEBAND_RESET renamed /FPGA Configuration and Dev Features/~{SIDEBAND_RESET}
- net /FPGA Configuration and Dev Features/~UC_RESET renamed /FPGA Configuration and Dev Features/~{UC_RESET}
- net /Host Section/~HOST_RESET renamed /Host Section/~{HOST_RESET}
- net /RAM Section/~RAM_CLK renamed /RAM Section/~{RAM_CLK}
- net /RAM Section/~RAM_CS renamed /RAM Section/~{RAM_CS}
- net /RAM Section/~RAM_RESET renamed /RAM Section/~{RAM_RESET}
- net /Target Section/~TARGET_RESET renamed /Target Section/~{TARGET_RESET}
Other:
- net class Default removed
- board text added: "powered by nMigen"
- board text removed: "powered by Amaranth HDL"
